File: hardware/pcb/single_channel_1G.kicad_sch (KiCad schematic)
At the start: 23 parts, among them J1 BNC (insect electrode), J2 Lemo/ODU 8-pin to motherboard, K1 latching reed relay (Ri sw), U3 ADA4940-1ARZ-RL, U4 latching-relay driver (H-brid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

Commit message: start 1G design
Parts:
- removed K1: latching reed relay (Ri sw), Relay_THT:Relay_1-Form-A_Schrack-RYII_RM5mm, symbol epg:K1
- removed U4: latching-relay driver (H-bridge), Package_TO_SOT_SMD:SOT-23-6, symbol epg:U4
- added J3: BNC (insect electrode), Connector_Coaxial:BNC_Amphenol_031-5539_Vertical, symbol epg:J1
- RI1: footprint Resistor_SMD:R_1206_3216Metric -> Resistor_THT:R_Axial_DIN0309_L9.0mm_D3.2mm_P20.32mm_Horizontal
Connections:
- net RI_MID is gone; now on an unnamed net: RI1.2
- net AGND: now also J3.2 (SHLD)
- net S: no longer A2.1 (+), RI1.1
- net M: no longer names the net of A1.1 (+), J1.1 (SIG)
- new net: A2.1 (+), J3.1 (SIG), RI1.1
Other:
- moved on the sheet: J1, RI1
