File: hardware/pcb/eagle/EPGinput.sch (EAGLE design)
At the start: 22 parts, among them J2 54-00248, J3 BNCPTH, U1 ADA4530-1, U2 ADA4530-1, U3 ADA4940-1

Commit message: Eagle PCB updates
Parts:
- removed J3: BNCPTH, SparkFun-Connectors:BNCPTH
- added J1: BNCBJ21, STEVES_BU:BNCBJ21
- R9: device resistor:R-US_0414/15 -> resistor:R-US_0617/22
Connections:
- net N$5 renamed SIGOUT
- net N$8 renamed VSOUT
- net GND: now also J1.GND@1; no longer J3.GND
- net N$2: now also J1.1; no longer J3.OUT
Changed lines of the file:
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@@
 <part name="C6" library="STEVES_BU" deviceset="CAPS" device="0603S"/>
 <part name="C7" library="STEVES_BU" deviceset="CAPS" device="0603S"/>
-<part name="R9" library="resistor" deviceset="R-US_" device="0414/15"/>
+<part name="R9" library="resistor" deviceset="R-US_" device="0617/22"/>
 <part name="GND1" library="SparkFun-PowerSymbols" deviceset="GND" device=""/>
 <part name="GND2" library="SparkFun-PowerSymbols" deviceset="GND" device=""/>
@@
 <part name="GND9" library="SparkFun-PowerSymbols" deviceset="GND" device=""/>
 <part name="J2" library="54-00248" deviceset="54-00248" device=""/>
-<part name="J3" library="SparkFun-Connectors" deviceset="BNC" device="PTH"/>
+<part name="J1" library="STEVES_BU" deviceset="BNC" device="BJ21"/>
 </parts>
 <sheets>
@@
 <instance part="GND9" gate="1" x="96.52" y="53.34"/>
 <instance part="J2" gate="G$1" x="124.46" y="58.42" rot="MR0"/>
-<instance part="J3" gate="G$1" x="-53.34" y="91.44"/>
+<instance part="J1" gate="G$1" x="-55.88" y="91.44"/>
 </instances>
 <busses>
@@
 </segment>
 </net>
-<net name="N$5" class="0">
+<net name="SIGOUT" class="0">
 <segment>
 <pinref part="U1" gate="G$1" pin="OUT"/>
@@
 <pinref part="R1" gate="G$1" pin="1"/>
 <wire x1="35.56" y1="71.12" x2="38.1" y2="71.12" width="0.1524" layer="91"/>
+<label x="20.32" y="88.9" size="1.778" layer="95"/>
 </segment>
 </net>
@@
 </segment>
 </net>
-<net name="N$8" class="0">
+<net name="VSOUT" class="0">
 <segment>
 <pinref part="U2" gate="G$1" pin="OUT"/>
@@
 <wire x1="15.24" y1="12.7" x2="15.24" y2="35.56" width="0.1524" layer="91"/>
 <junction x="15.24" y="35.56"/>
+<label x="22.86" y="38.1" size="1.778" layer="95"/>
 </segment>
 </net>
@@
 </segment>
 <segment>
-<pinref part="GND8" gate="1" pin="GND"/>
-<pinref part="J3" gate="G$1" pin="GND"/>
-</segment>
-<segment>
 <pinref part="GND9" gate="1" pin="GND"/>
 <wire x1="114.3" y1="55.88" x2="96.52" y2="55.88" width="0.1524" layer="91"/>
 <pinref part="J2" gate="G$1" pin="6"/>
+</segment>
+<segment>
+<pinref part="J1" gate="G$1" pin="GND@1"/>
+<pinref part="GND8" gate="1" pin="GND"/>
+<wire x1="-53.34" y1="88.9" x2="-53.34" y2="86.36" width="0.1524" layer="91"/>
 </segment>
 </net>
@@
 <wire x1="-35.56" y1="91.44" x2="-35.56" y2="68.58" width="0.1524" layer="91"/>
 <pinref part="R9" gate="G$1" pin="2"/>
-<wire x1="-35.56" y1="91.44" x2="-48.26" y2="91.44" width="0.1524" layer="91"/>
+<wire x1="-35.56" y1="91.44" x2="-53.34" y2="91.44" width="0.1524" layer="91"/>
 <junction x="-35.56" y="91.44"/>
-<pinref part="J3" gate="G$1" pin="OUT"/>
-</segment>
-</net>
+<pinref part="J1" gate="G$1" pin="1"/>
+</segment>
+</net>

Commit message: board out
Parts:
- removed J2: 54-00248, 54-00248:54-00248
- removed R9: (no value), resistor:R-US_0617/22
- added C10: 0.1, STEVES_BU:CAPS0603S
- added C9: 10, STEVES_BU:CAPS1206S
- added GRD, SHIELD, VS: (no value), wirepad:2,15/1,0
- added IN: (no value), wirepad:SMD2
- C6: value (none) -> 10; device STEVES_BU:CAPS0603S -> STEVES_BU:CAPS1206S
- J1: value BNCBJ21 -> 54-00248; device STEVES_BU:BNCBJ21 -> 54-00248:54-00248
Connections:
- removed net -5V: C7.2, U3.V-
- removed net N$2: J1.1, R9.2, U1.+IN
- removed net N$3: U1.GRD1, U1.GRD2
- new net GUARD: GRD.P, U1.GRD1, U1.GRD2
- new net PROBE: IN.P, U1.+IN
- net -5V0: now also C6.1, C7.2, J1.5, U3.V-; no longer J2.5
- net 5V0: now also C9.1, J1.4; no longer J2.4
- net GND: now also C10.2, C6.2, C9.2, J1.6; no longer J1.GND@1, J2.6
- net N$10: now also J1.1; no longer J2.1
- net N$9: now also J1.2; no longer J2.2
- net SHIELD: now also J1.8, J1.SHELL, SHIELD.P; no longer J2.8, J2.SHELL
- net VS: now also C10.1, J1.7, VS.P; no longer J2.7, R9.1
Other:
- moved on the sheet: C6

Commit message: started control board
Parts:
- R1, R2, R8: value (none) -> 1K00
- R3, R4: value (none) -> 24R
- R5, R6: value (none) -> 8K06
- R7: value (none) -> 2K00
