File: hardware/pcb/eagle/EPGinputRelay.sch (EAGLE design)
At the start: 26 parts, among them J1 54-00248, U1 ADA4530-1, U2 ADA4530-1, U3 ADA4940-1

Commit message: PCB w/ relay
Parts:
- removed RL1: REED-RELAY, EPGinput:REED-RELAY
- added K1: REED-RELAY, EPGinput:REED-RELAY
- added VS: (no value), wirepad:2,15/1,0
- C10: value 0.1 -> (none)
- C2: value (none) -> 0.1
- C4, C8: value (none) -> 10; device STEVES_BU:CAPS0603S -> STEVES_BU:CAPS1206S
- C6, C9: value 10 -> (none); device STEVES_BU:CAPS1206S -> STEVES_BU:CAPS0603S
- IN: device wirepad:SMD2 -> jETPAK-ASM:PADPAD150
- U2: value ADA4530-1 -> ADA4940-1; device EPG:ADA4530-1 -> EPG:ADA4940-1
- U3: value ADA4940-1 -> ADA4530-1; device EPG:ADA4940-1 -> EPG:ADA4530-1
Connections:
- removed net N$1: C2.1, R7.1, R8.2, U3.VOCM
- removed net RLY: J1.3, RL1.C2
- removed net SHIELD: J1.8, J1.SHELL, SHIELD.P
- new net N$2: J1.SHELL, SHIELD.P
- new net RLY+: J1.3, K1.C2
- new net RLY-: J1.8, K1.C1
- new net VCOM: C1.1, R1.2, R4.1, U2.VOCM
- net -5V0: now also C3.1, U3.IC; no longer C5.1, U2.IC
- net 5V0: now also C10.1, C5.1, C8.1, C9.2, R4.2, U2.EN; no longer C1.1, C3.1, C8.2, C9.1, R7.2, U3.EN
- net GND: now also C8.2, C9.1, R1.1; no longer C8.1, C9.2, R8.1, RL1.C1
- net GUARD: now also K1.GRD, U3.GRD1, U3.GRD2; no longer RL1.GRD, U1.GRD1, U1.GRD2
- net N$10: now also R2.2; no longer R4.2
- net N$19: now also R2.1, R3.2, U2.+OUT; no longer R4.1, R5.2, U3.+OUT
- net N$20: now also R6.1, R7.2, U2.-OUT; no longer R3.1, R6.2, U3.-OUT
- net N$6: now also R7.1, R8.2, U2.+IN; no longer R1.2, R6.1, U3.+IN
- net N$7: now also R3.1, R5.2, U2.-IN; no longer R2.2, R5.1, U3.-IN
- net N$9: now also R6.2; no longer R3.2
- net PROBE: now also IN.1, U3.+IN; no longer IN.P, U1.+IN
- net SIGOUT: now also R8.1, U3.-IN, U3.OUT; no longer R1.1, U1.-IN, U1.OUT
- net VS: now also C2.1, U1.+IN, VS.P; no longer C10.1, U2.+IN
- net VSOUT: now also R5.1, U1.-IN, U1.OUT; no longer R2.1, U2.-IN, U2.OUT
Other:
- moved on the sheet: C1, C10, C2, C3, C4, C5, C6, C8, C9, GD, R1, R2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

Commit message: started control board
Connections:
- net N$10 renamed AOP\
- net N$9 renamed AON
Changed lines of the file:
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@@
 <grid distance="0.1" unitdist="inch" unit="inch" style="lines" multiple="1" display="no" altdistance="0.01" altunitdist="inch" altunit="inch"/>
 <layers>
-<layer number="1" name="Top" color="4" fill="1" visible="yes" active="no"/>
-<layer number="2" name="Route2" color="1" fill="3" visible="yes" active="no"/>
-<layer number="3" name="Route3" color="4" fill="3" visible="yes" active="no"/>
-<layer number="4" name="Route4" color="1" fill="4" visible="yes" active="no"/>
-<layer number="5" name="Route5" color="4" fill="4" visible="yes" active="no"/>
-<layer number="6" name="Route6" color="1" fill="8" visible="yes" active="no"/>
-<layer number="7" name="Route7" color="4" fill="8" visible="yes" active="no"/>
-<layer number="8" name="Route8" color="1" fill="2" visible="yes" active="no"/>
-<layer number="9" name="Route9" color="4" fill="2" visible="yes" active="no"/>
-<layer number="10" name="Route10" color="1" fill="7" visible="yes" active="no"/>
-<layer number="11" name="Route11" color="4" fill="7" visible="yes" active="no"/>
-<layer number="12" name="Route12" color="1" fill="5" visible="yes" active="no"/>
-<layer number="13" name="Route13" color="4" fill="5" visible="yes" active="no"/>
-<layer number="14" name="Route14" color="1" fill="6" visible="yes" active="no"/>
-<layer number="15" name="Route15" color="4" fill="6" visible="yes" active="no"/>
-<layer number="16" name="Bottom" color="1" fill="1" visible="yes" active="no"/>
-<layer number="17" name="Pads" color="2" fill="1" visible="yes" active="no"/>
-<layer number="18" name="Vias" color="2" fill="1" visible="yes" active="no"/>
-<layer number="19" name="Unrouted" color="6" fill="1" visible="yes" active="no"/>
-<layer number="20" name="Dimension" color="15" fill="1" visible="yes" active="no"/>
-<layer number="21" name="tPlace" color="7" fill="1" visible="yes" active="no"/>
-<layer number="22" name="bPlace" color="7" fill="1" visible="yes" active="no"/>
-<layer number="23" name="tOrigins" color="15" fill="1" visible="yes" active="no"/>
-<layer number="24" name="bOrigins" color="15" fill="1" visible="yes" active="no"/>
-<layer number="25" name="tNames" color="7" fill="1" visible="yes" active="no"/>
-<layer number="26" name="bNames" color="7" fill="1" visible="yes" active="no"/>
-<layer number="27" name="tValues" color="7" fill="1" visible="yes" active="no"/>
-<layer number="28" name="bValues" color="7" fill="1" visible="yes" active="no"/>
+<layer number="1" name="Top" color="4" fill="1" visible="no" active="no"/>
+<layer number="2" name="Route2" color="1" fill="3" visible="no" active="no"/>
+<layer number="3" name="Route3" color="4" fill="3" visible="no" active="no"/>
+<layer number="4" name="Route4" color="1" fill="4" visible="no" active="no"/>
+<layer number="5" name="Route5" color="4" fill="4" visible="no" active="no"/>
+<layer number="6" name="Route6" color="1" fill="8" visible="no" active="no"/>
+<layer number="7" name="Route7" color="4" fill="8" visible="no" active="no"/>
+<layer number="8" name="Route8" color="1" fill="2" visible="no" active="no"/>
+<layer number="9" name="Route9" color="4" fill="2" visible="no" active="no"/>
+<layer number="10" name="Route10" color="1" fill="7" visible="no" active="no"/>
+<layer number="11" name="Route11" color="4" fill="7" visible="no" active="no"/>
+<layer number="12" name="Route12" color="1" fill="5" visible="no" active="no"/>
+<layer number="13" name="Route13" color="4" fill="5" visible="no" active="no"/>
+<layer number="14" name="Route14" color="1" fill="6" visible="no" active="no"/>
+<layer number="15" name="Route15" color="4" fill="6" visible="no" active="no"/>
+<layer number="16" name="Bottom" color="1" fill="1" visible="no" active="no"/>
+<layer number="17" name="Pads" color="2" fill="1" visible="no" active="no"/>
+<layer number="18" name="Vias" color="2" fill="1" visible="no" active="no"/>
+<layer number="19" name="Unrouted" color="6" fill="1" visible="no" active="no"/>
+<layer number="20" name="Dimension" color="15" fill="1" visible="no" active="no"/>
+<layer number="21" name="tPlace" color="7" fill="1" visible="no" active="no"/>
+<layer number="22" name="bPlace" color="7" fill="1" visible="no" active="no"/>
+<layer number="23" name="tOrigins" color="15" fill="1" visible="no" active="no"/>
+<layer number="24" name="bOrigins" color="15" fill="1" visible="no" active="no"/>
+<layer number="25" name="tNames" color="7" fill="1" visible="no" active="no"/>
+<layer number="26" name="bNames" color="7" fill="1" visible="no" active="no"/>
+<layer number="27" name="tValues" color="7" fill="1" visible="no" active="no"/>
+<layer number="28" name="bValues" color="7" fill="1" visible="no" active="no"/>
 <layer number="29" name="tStop" color="7" fill="3" visible="no" active="no"/>
 <layer number="30" name="bStop" color="7" fill="6" visible="no" active="no"/>
@@
 <layer number="35" name="tGlue" color="7" fill="4" visible="no" active="no"/>
 <layer number="36" name="bGlue" color="7" fill="5" visible="no" active="no"/>
-<layer number="37" name="tTest" color="7" fill="1" visible="yes" active="no"/>
-<layer number="38" name="bTest" color="7" fill="1" visible="yes" active="no"/>
+<layer number="37" name="tTest" color="7" fill="1" visible="no" active="no"/>
+<layer number="38" name="bTest" color="7" fill="1" visible="no" active="no"/>
 <layer number="39" name="tKeepout" color="4" fill="11" visible="no" active="no"/>
 <layer number="40" name="bKeepout" color="1" fill="11" visible="no" active="no"/>
@@
 <layer number="44" name="Drills" color="7" fill="1" visible="no" active="no"/>
 <layer number="45" name="Holes" color="7" fill="1" visible="no" active="no"/>
-<layer number="46" name="Milling" color="3" fill="1" visible="yes" active="no"/>
-<layer number="47" name="Measures" color="7" fill="1" visible="yes" active="no"/>
-<layer number="48" name="Document" color="7" fill="1" visible="yes" active="no"/>
-<layer number="49" name="Reference" color="7" fill="1" visible="yes" active="no"/>
-<layer number="50" name="dxf" color="7" fill="1" visible="yes" active="no"/>
-<layer number="51" name="tDocu" color="7" fill="1" visible="yes" active="no"/>
-<layer number="52" name="bDocu" color="7" fill="1" visible="yes" active="no"/>
-<layer number="53" name="tGND_GNDA" color="7" fill="9" visible="yes" active="no"/>
-<layer number="54" name="bGND_GNDA" color="1" fill="9" visible="yes" active="no"/>
-<layer number="56" name="wert" color="7" fill="1" visible="yes" active="no"/>
-<layer number="57" name="tCAD" color="7" fill="1" visible="yes" active="no"/>
-<layer number="58" name="b3D" color="7" fill="1" visible="yes" active="no"/>
-<layer number="59" name="tCarbon" color="7" fill="1" visible="yes" active="no"/>
-<layer number="60" name="bCarbon" color="7" fill="1" visible="yes" active="no"/>
-<layer number="61" name="stand" color="7" fill="1" visible="yes" active="no"/>
+<layer number="46" name="Milling" color="3" fill="1" visible="no" active="no"/>
+<layer number="47" name="Measures" color="7" fill="1" visible="no" active="no"/>
+<layer number="48" name="Document" color="7" fill="1" visible="no" active="no"/>
+<layer number="49" name="Reference" color="7" fill="1" visible="no" active="no"/>
+<layer number="50" name="dxf" color="7" fill="1" visible="no" active="no"/>
+<layer number="51" name="tDocu" color="7" fill="1" visible="no" active="no"/>
+<layer number="52" name="bDocu" color="7" fill="1" visible="no" active="no"/>
+<layer number="53" name="tGND_GNDA" color="7" fill="9" visible="no" active="no"/>
+<layer number="54" name="bGND_GNDA" color="1" fill="9" visible="no" active="no"/>
+<layer number="56" name="wert" color="7" fill="1" visible="no" active="no"/>
+<layer number="57" name="tCAD" color="7" fill="1" visible="no" active="no"/>
+<layer number="58" name="b3D" color="7" fill="1" visible="no" active="no"/>
+<layer number="59" name="tCarbon" color="7" fill="1" visible="no" active="no"/>
+<layer number="60" name="bCarbon" color="7" fill="1" visible="no" active="no"/>
+<layer number="61" name="stand" color="7" fill="1" visible="no" active="no"/>
 <layer number="88" name="SimResults" color="7" fill="1" visible="yes" active="yes"/>
 <layer number="89" name="SimProbes" color="7" fill="1" visible="yes" active="yes"/>
@@
 <wire x1="114.3" y1="55.88" x2="96.52" y2="55.88" width="0.1524" layer="91"/>
 <pinref part="J1" gate="1" pin="6"/>
+<label x="106.68" y="55.88" size="1.778" layer="95"/>
 </segment>
 <segment>
@@
 <segment>
 <wire x1="114.3" y1="53.34" x2="104.14" y2="53.34" width="0.1524" layer="91"/>
-<label x="106.68" y="53.34" size="1.778" layer="95"/>
+<label x="109.22" y="53.34" size="1.778" layer="95"/>
 <pinref part="J1" gate="1" pin="7"/>
 </segment>
@@
 <segment>
 <wire x1="114.3" y1="50.8" x2="111.76" y2="50.8" width="0.1524" layer="91"/>
-<label x="101.6" y="50.8" size="1.778" layer="95"/>
+<label x="109.22" y="50.8" size="1.778" layer="95"/>
 <wire x1="111.76" y1="50.8" x2="101.6" y2="50.8" width="0.1524" layer="91"/>
 <pinref part="J1" gate="1" pin="8"/>
@@
 </segment>
 </net>
-<net name="N$9" class="0">
+<net name="AON" class="0">
 <segment>
 <pinref part="R6" gate="G$1" pin="2"/>
@@
 <wire x1="101.6" y1="66.04" x2="101.6" y2="68.58" width="0.1524" layer="91"/>
 <pinref part="J1" gate="1" pin="2"/>
-</segment>
-</net>
-<net name="N$10" class="0">
+<label x="106.68" y="66.04" size="1.778" layer="95"/>
+</segment>
+</net>
+<net name="AOP\" class="0">
 <segment>
 <pinref part="R2" gate="G$1" pin="2"/>
@@
 <wire x1="104.14" y1="68.58" x2="114.3" y2="68.58" width="0.1524" layer="91"/>
 <pinref part="J1" gate="1" pin="1"/>
-</segment>
-</net>
+<label x="106.68" y="68.58" size="1.778" layer="95"/>
+</segment>
+</net>
