File: hardware/pcb/eagle/EPGcontrol.brd (EAGLE design)
At the start: 228.6 x 101.6 mm, 12 parts, among them IC1 ADS131M08QPBSRQ1, J1 54-00248, J2 54-00248, J3 54-00248, J4 54-00248, J5 54-00248, J6 54-00248, J7 54-00248, J8 54-00248, U1 DAC8568IBPW

Commit message: Control Board updates
Parts:
- added C1, C2, C3, C4, C5, C6, C7, C8: 4.7n, STEVES_BU:0603S
- added C10, C16, C18, C19, C23: 10u, rcl:C1206
- added C11, C12, C13, C14, C15, C20, C21, C9: 0.1u, STEVES_BU:0603S
- added C24, C26: 47, rcl:C1206
- added D1, D2: (no value), SparkFun:SMA-DIODE
- added L1, L2: FERRITE BEAD, STEVES_BU:0805S
- added R1, R10, R11, R12, R13, R14, R15, R16, R2, R3, R4, R5, R6, R7, R8, R9: 49R9, STEVES_BU:0805S
- added R17: 102K, rcl:R0805
- added R18: 332K, rcl:R0805
- added U4: TPS7A470X, STEVES_BU:VQFN-20-5X5
- added U5: TPS7A33, STEVES_BU:VQFN-20-5X5
- PS1: value LM27762DSSR -> NMH0509DC; device SamacSys_Parts:SON50P200X300X80-13N -> STEVES_BU:PDM2
- moved PS1 128.0 mm to (211.4, 70.7), turned to 270 degrees
- moved U$1 1.70 mm to (106.4, 66.5)
- renumbered IC1 to U2
Connections:
- removed net AVDD: U1.3
- removed net C1+: PS1.10
- removed net C1-: PS1.9
- removed net CP: PS1.5
- removed net FB+: PS1.2
- removed net FB-: PS1.7
- removed net OUT+: PS1.11
- removed net OUT-: PS1.6
- removed net PAD: PS1.13
- removed net VIN: PS1.3
- new net +9V: C19.1, C21.1, L2.1, PS1.9
- new net -9V: C18.2, C20.2, L1.1, PS1.11
- new net ADCCLK: U2.23
- new net ADCCS: U2.17
- new net ADCRDY: U2.18
- new net AGND: C12.2, C13.2, C14.2, C24.2, C26.2, D1.A, D2.C, J1.6, J2.6, J3.6, J4.6, J5.6, J6.6, J7.6, J8.6, R17.1, U1.14, U2.13, U2.28, U4.P$10, U4.P$6, U4.P$7, U4.PAD1, U4.PAD2, U4.PAD3, U4.PAD4, U4.PAD5, U4.PAD6, U4.PAD7, U4.PAD8, U4.PAD9, U5.P$7, U5.PAD1, U5.PAD2, U5.PAD3, U5.PAD4, U5.PAD5, U5.PAD6, U5.PAD7, U5.PAD8, U5.PAD9
- new net AIN0N: J1.2, R16.1
- new net AIN0P: J1.1, R15.1
- new net AIN1N: J2.2, R12.1
- new net AIN1P: J2.1, R11.1
- new net AIN2N: J3.2, R8.1
- new net AIN2P: J3.1, R7.1
- new net AIN3N: J4.2, R6.1
- new net AIN3P: J4.1, R5.1
- new net AIN4N: J5.2, R2.1
- new net AIN4P: J5.1, R1.1
- new net AIN5N: J6.1, R13.1
- new net AIN5P: J6.2, R14.1
- new net AIN6N: J7.2, R10.1
- new net AIN6P: J7.1, R9.1
- new net AIN7N: J8.2, R4.1
- new net AIN7P: J8.1, R3.1
- new net N$1: C15.2, R17.2, R18.1, U5.P$3
- new net N$10: U1.8
- new net N$18: C13.1, U5.P$14
- new net N$23: C12.1, U4.P$14
- new net N$4: U1.2
- new net N$5: U1.1
- new net N$9: U1.9
- new net SPICS: U$1.22
- new net SPIOCLK: U$1.24, U1.16, U2.19
- new net SPIORX: U$1.21, U2.20
- new net SPIOTX: U$1.25, U1.15, U2.21
- new net USB+: C23.1, PS1.14
- new net USB-: C23.2, PS1.1
- new net VIN+: C10.1, C9.1, L2.2, U4.P$13, U4.P$15, U4.P$16
- new net VIN-: C11.1, C16.1, L1.2, U5.P$13, U5.P$15, U5.P$16
- net -5V0: now also C15.1, C26.1, D2.A, R18.2, U5.P$1, U5.P$20
- net 5V0: now also C14.1, C24.1, D1.C, U1.3, U2.15, U4.P$1, U4.P$20, U4.P$3
- net A0N: now also C8.2, R16.2; no longer J1.2
- net A0P: now also C8.1, R15.2; no longer J1.1
- net A1N: now also C6.2, R12.2; no longer J2.2
- net A1P: now also C6.1, R11.2; no longer J2.1
- net A2N: now also C4.2, R8.2; no longer J3.2
- net A2P: now also C4.1, R7.2; no longer J3.1
- net A3N: now also C3.2, R6.2; no longer J4.2
- net A3P: now also C3.1, R5.2; no longer J4.1
- net A4N: now also C1.2, R2.2; no longer J5.2
- net A4P: now also C1.1, R1.2; no longer J5.1
- net A5N: now also C7.2, R14.2; no longer J6.2
- net A5P: now also C7.1, R13.2; no longer J6.1
- net A6N: now also C5.2, R10.2; no longer J7.2
- net A6P: now also C5.1, R9.2; no longer J7.1
- net A7N: now also C2.2, R4.2; no longer J8.2
- net A7P: now also C2.1, R3.2; no longer J8.1
- net GND: now also C10.2, C11.2, C16.2, C18.1, C19.2, C20.1, C21.2, C9.2, PS1.8, U$1.13, U$1.18, U$1.23, U$1.28, U$1.3, U$1.33, U$1.38, U$1.8, U$1.GND, U2.25; no longer J1.6, J2.6, J3.6, J4.6, J5.6, J6.6, J7.6, J8.6, PS1.4, U1.14
Routing:
- net -5V0: track 0.00 -> 292.0 mm, vias 0 -> 1
- net 5V0: track 0.00 -> 291.1 mm
- net SPIOTX: track 0.00 -> 44.8 mm, vias 0 -> 2
- net VIN+: track 0.00 -> 40.5 mm
- net AGND: track 0.00 -> 40.0 mm, vias 0 -> 15
- net SPIOCLK: track 0.00 -> 38.9 mm, vias 0 -> 2
- net VIN-: track 0.00 -> 35.7 mm
- net VS3: track 54.2 -> 29.4 mm, vias 0 -> 2
- net +9V: track 0.00 -> 24.2 mm, vias 0 -> 1
- net VS1: track 103.1 -> 81.4 mm, vias 0 -> 6
- net -9V: track 0.00 -> 20.9 mm
- net VS2: track 69.9 -> 51.9 mm, vias 1 -> 4
- net GND: track 0.00 -> 15.8 mm, vias 0 -> 9
- net VS0: track 112.0 -> 98.4 mm, vias 0 -> 7
- net VS6: track 88.1 -> 75.7 mm, vias 2 -> 4
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- added copper zone on layer 16, net AGND
- added copper zone on layer 16, net GND
Other:
- board size 228.6 x 101.6 mm -> 228.6 x 92.5 mm

Commit message: updates to controller
Parts:
- added J10, J11, J12, J9: FCR7350G, STEVES_BU:CONN_FCR7350G_CLF
- C10, C16, C18, C19, C23: value 10u -> 10
- C11, C12, C13, C14, C15, C20, C21, C9: value 0.1u -> 0.1
Routing:
- net 5V0: track 291.1 -> 423.3 mm, vias 0 -> 4
- net AGND: track 40.0 -> 40.5 mm

Commit message: EPGcontrol PCB updates - relay
Parts:
- added C17: 220n, STEVES_BU:0603S
- added C22: 150n, STEVES_BU:0603S
- added C25, C27: 10, STEVES_BU:1206S
- added D3, D4: DIODE, SparkFun-DiscreteSemi:SOD-323
- added Q1, Q2: 2N3904, SparkFun-DiscreteSemi:SOT23-3
- added R19, R20, R21, R22: 1K00, STEVES_BU:0805S
- moved D1 6.65 mm to (219.6, 18.6)
- moved C24 6.65 mm to (219.4, 22.6)
- moved C26 6.04 mm to (210.6, 22.2), turned to 180 degrees
- moved D2 5.09 mm to (210.7, 19.2)
- moved C13 3.39 mm to (200.4, 31.3)
- moved C15 3.39 mm to (209.1, 25.7)
- moved R17 3.39 mm to (211.1, 29.6)
- moved R18 3.39 mm to (211.3, 25.6)
- moved U5 3.39 mm to (204.1, 28.7)
- moved C12 2.96 mm to (224.4, 29.5)
- moved U4 2.96 mm to (219.9, 28.5)
- moved C14 2.96 mm to (215.1, 28.8)
Connections:
- removed net N$5: U1.1
- removed net N$9: U1.9
- new net 5VD: C25.1, C27.1, R19.2, R20.2
- new net ADCSYNC: U$1.29, U2.16
- new net DACCS: U$1.17, U1.2
- new net DACRST: U$1.20, U1.9
- new net LDAC: U$1.19, U1.1
- new net N$2: C17.1, U2.24
- new net N$3: Q2.1, R21.1
- new net R6: R21.2, U$1.32
- new net R7: R22.2, U$1.31
- new net RGND: Q1.2, Q2.2
- net ADCCLK: now also U$1.27
- net ADCRDY: now also U$1.26
- net AGND: now also C22.2
- net GND: now also C17.2
- net K6N: now also D4.A, Q2.3
- net K6P: now also C27.2, D4.C, R20.1
- net K7N: now also D3.A, Q1.3
- net K7P: now also C25.2, D3.C, R19.1
- net N$10: now also C22.1
- net N$4: now also Q1.1, R22.1; no longer U1.2
Routing:
- net R6: track 0.00 -> 90.5 mm, vias 0 -> 2
- net 5VD: track 0.00 -> 61.1 mm, vias 0 -> 4
- net RGND: track 0.00 -> 49.0 mm, vias 0 -> 4
- net DACCS: track 0.00 -> 32.6 mm, vias 0 -> 2
- net DACRST: track 0.00 -> 32.6 mm, vias 0 -> 2
- net ADCSYNC: track 0.00 -> 30.8 mm, vias 0 -> 2
- net ADCCLK: track 0.00 -> 28.4 mm, vias 0 -> 1
- net LDAC: track 0.00 -> 25.7 mm, vias 0 -> 2
- net ADCRDY: track 0.00 -> 22.5 mm, vias 0 -> 2
- net R7: track 0.00 -> 22.5 mm, vias 0 -> 2
- net K7P: track 0.00 -> 14.3 mm
- net K6N: track 0.00 -> 14.3 mm
- net K6P: track 0.00 -> 14.0 mm, vias 0 -> 1
- net K7N: track 0.00 -> 13.4 mm, vias 0 -> 1
- net +9V: track 24.2 -> 17.3 mm, vias 1 -> 0
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