File: hardware/pcb/eagle/EPGcontrol.sch (EAGLE design)
At the start: 12 parts, among them IC1 ADS131M08QPBSRQ1, J1 54-00248, J2 54-00248, J3 54-00248, J4 54-00248, J5 54-00248, J6 54-00248, J7 54-00248, J8 54-00248, U1 DAC8568IBPW

Commit message: Control Board updates
Parts:
- removed IC1: ADS131M08QPBSRQ1, SamacSys_Parts:ADS131M08QPBSRQ1
- added C1, C2, C3, C4, C5, C6, C7, C8: 4.7n, STEVES_BU:CAPS0603S
- added C10, C16, C18, C19, C23: 10u, rcl:C-EUC1206
- added C11, C12, C13, C14, C15, C20, C21, C9: 0.1u, STEVES_BU:CAPS0603S
- added C24, C26: 47, rcl:C-EUC1206
- added D1, D2: (no value), SparkFun:DIODESMA
- added L1, L2: FERRITE BEAD, STEVES_BU:INDUCTOR_SM0805S
- added R1, R10, R11, R12, R13, R14, R15, R16, R2, R3, R4, R5, R6, R7, R8, R9: 49R9, STEVES_BU:RESISTOR_SM0805S
- added R17: 102K, rcl:R-US_R0805
- added R18: 332K, rcl:R-US_R0805
- added U2: ADS131M08QPBSRQ1, SamacSys_Parts:ADS131M08QPBSRQ1
- added U4: TPS7A470X, STEVES_BU:TPS7A470X
- added U5: TPS7A33, STEVES_BU:TPS7A33
- PS1: value LM27762DSSR -> NMH0509DC; device SamacSys_Parts:LM27762DSSR -> STEVES_BU:DC-DC-PDS1-DUALPDM2
Connections:
- new net +9V: C19.1, C21.1, L2.1, PS1.+VO
- new net -9V: C18.2, C20.2, L1.1, PS1.-VO
- new net ADCCLK: U2.XTAL1/CLKIN
- new net ADCCS: U2.!CS
- new net ADCRDY: U2.!DRDY
- new net AGND: C12.2, C13.2, C14.2, C24.2, C26.2, D1.A, D2.C, J1.6, J2.6, J3.6, J4.6, J5.6, J6.6, J7.6, J8.6, R17.1, U2.AGND_1, U2.AGND_2, U4.3P2V, U4.GND, U4.OP4V, U5.GND
- new net AIN0N: J1.2, R16.1
- new net AIN0P: J1.1, R15.1
- new net AIN1N: J2.2, R12.1
- new net AIN1P: J2.1, R11.1
- new net AIN2N: J3.2, R8.1
- new net AIN2P: J3.1, R7.1
- new net AIN3N: J4.2, R6.1
- new net AIN3P: J4.1, R5.1
- new net AIN4N: J5.2, R2.1
- new net AIN4P: J5.1, R1.1
- new net AIN5N: J6.1, R13.1
- new net AIN5P: J6.2, R14.1
- new net AIN6N: J7.2, R10.1
- new net AIN6P: J7.1, R9.1
- new net AIN7N: J8.2, R4.1
- new net AIN7P: J8.1, R3.1
- new net N$1: C15.2, R17.2, R18.1, U5.FB
- new net N$10: U1.VREFIN/OUT
- new net N$18: C13.1, U5.NR
- new net N$23: C12.1, U4.NR
- new net N$4: U1.!SYNC
- new net N$5: U1.!LDAC
- new net N$9: U1.!CLR
- new net SPICS: U$1.17/SPCS
- new net SPIOCLK: U$1.18/SPCK, U1.SCLK, U2.SCLK
- new net SPIORX: U$1.16/SPRX, U2.DOUT
- new net SPIOTX: U$1.19/SPTX, U1.DIN, U2.DIN
- new net USB+: C23.1, PS1.VIN
- new net USB-: C23.2, PS1.GND
- new net VIN+: C10.1, C9.1, L2.2, U4.EN, U4.IN1, U4.IN2
- new net VIN-: C11.1, C16.1, L1.2, U5.EN, U5.IN1, U5.IN2
- net -5V0: now also C15.1, C26.1, D2.A, R18.2, U5.OUT1, U5.OUT2
- net 5V0: now also C14.1, C24.1, D1.C, U1.AVDD, U2.AVDD, U4.OUT1, U4.OUT2, U4.SENSE
- net A0N: now also C8.2, R16.2, U2.AIN0N; no longer IC1.AIN0N, J1.2
- net A0P: now also C8.1, R15.2, U2.AIN0P; no longer IC1.AIN0P, J1.1
- net A1N: now also C6.2, R12.2, U2.AIN1N; no longer IC1.AIN1N, J2.2
- net A1P: now also C6.1, R11.2, U2.AIN1P; no longer IC1.AIN1P, J2.1
- net A2N: now also C4.2, R8.2, U2.AIN2N; no longer IC1.AIN2N, J3.2
- net A2P: now also C4.1, R7.2, U2.AIN2P; no longer IC1.AIN2P, J3.1
- net A3N: now also C3.2, R6.2, U2.AIN3N; no longer IC1.AIN3N, J4.2
- net A3P: now also C3.1, R5.2, U2.AIN3P; no longer IC1.AIN3P, J4.1
- net A4N: now also C1.2, R2.2, U2.AIN4N; no longer IC1.AIN4N, J5.2
- net A4P: now also C1.1, R1.2, U2.AIN4P; no longer IC1.AIN4P, J5.1
- net A5N: now also C7.2, R14.2, U2.AIN5N; no longer IC1.AIN5N, J6.2
- net A5P: now also C7.1, R13.2, U2.AIN5P; no longer IC1.AIN5P, J6.1
- net A6N: now also C5.2, R10.2, U2.AIN6N; no longer IC1.AIN6N, J7.2
- net A6P: now also C5.1, R9.2, U2.AIN6P; no longer IC1.AIN6P, J7.1
- net A7N: now also C2.2, R4.2, U2.AIN7N; no longer IC1.AIN7N, J8.2
- net A7P: now also C2.1, R3.2, U2.AIN7P; no longer IC1.AIN7P, J8.1
- net GND: now also C10.2, C11.2, C16.2, C18.1, C19.2, C20.1, C21.2, C9.2, PS1.0V, U$1.GND, U$1.GND1, U$1.GND2, U$1.GND3, U$1.GND4, U$1.GND5, U$1.GND6, U$1.GND7, U$1.GND8, U2.DGND; no longer J1.6, J2.6, J3.6, J4.6, J5.6, J6.6, J7.6, J8.6
Other:
- moved on the sheet: J1, J2, J3, J4, J5, J6, J7, J8, U1

Commit message: updates to controller
Parts:
- added J10, J11, J12, J9: FCR7350G, STEVES_BU:FCR7350G
- C10, C16, C18, C19, C23: value 10u -> 10
- C11, C12, C13, C14, C15, C20, C21, C9: value 0.1u -> 0.1
Changed lines of the file:
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@@
 <part name="C8" library="STEVES_BU" deviceset="CAPS" device="0603S" value="4.7n"/>
 <part name="U$1" library="pipico" deviceset="RASPBERRY-PI-PICO_TH" device=""/>
-<part name="C10" library="rcl" deviceset="C-EU" device="C1206" value="10u"/>
+<part name="C10" library="rcl" deviceset="C-EU" device="C1206" value="10"/>
 <part name="L2" library="STEVES_BU" deviceset="INDUCTOR_SM" device="0805S" value="FERRITE BEAD"/>
 <part name="L1" library="STEVES_BU" deviceset="INDUCTOR_SM" device="0805S" value="FERRITE BEAD"/>
 <part name="GND3" library="supply1" deviceset="GND" device=""/>
-<part name="C9" library="STEVES_BU" deviceset="CAPS" device="0603S" value="0.1u"/>
-<part name="C11" library="STEVES_BU" deviceset="CAPS" device="0603S" value="0.1u"/>
-<part name="C23" library="rcl" deviceset="C-EU" device="C1206" value="10u"/>
+<part name="C9" library="STEVES_BU" deviceset="CAPS" device="0603S" value="0.1"/>
+<part name="C11" library="STEVES_BU" deviceset="CAPS" device="0603S" value="0.1"/>
+<part name="C23" library="rcl" deviceset="C-EU" device="C1206" value="10"/>
 <part name="PS1" library="STEVES_BU" deviceset="DC-DC-PDS1-DUAL" device="PDM2" value="NMH0509DC"/>
 <part name="U4" library="STEVES_BU" deviceset="TPS7A470X" device=""/>
@@
 <part name="R17" library="rcl" deviceset="R-US_" device="R0805" value="102K"/>
 <part name="R18" library="rcl" deviceset="R-US_" device="R0805" value="332K"/>
-<part name="C12" library="STEVES_BU" deviceset="CAPS" device="0603S" value="0.1u"/>
-<part name="C13" library="STEVES_BU" deviceset="CAPS" device="0603S" value="0.1u"/>
-<part name="C14" library="STEVES_BU" deviceset="CAPS" device="0603S" value="0.1u"/>
-<part name="C15" library="STEVES_BU" deviceset="CAPS" device="0603S" value="0.1u"/>
-<part name="C16" library="rcl" deviceset="C-EU" device="C1206" value="10u"/>
+<part name="C12" library="STEVES_BU" deviceset="CAPS" device="0603S" value="0.1"/>
+<part name="C13" library="STEVES_BU" deviceset="CAPS" device="0603S" value="0.1"/>
+<part name="C14" library="STEVES_BU" deviceset="CAPS" device="0603S" value="0.1"/>
+<part name="C15" library="STEVES_BU" deviceset="CAPS" device="0603S" value="0.1"/>
+<part name="C16" library="rcl" deviceset="C-EU" device="C1206" value="10"/>
 <part name="GND12" library="supply1" deviceset="GND" device=""/>
 <part name="GND13" library="supply1" deviceset="GND" device=""/>
-<part name="C19" library="rcl" deviceset="C-EU" device="C1206" value="10u"/>
-<part name="C18" library="rcl" deviceset="C-EU" device="C1206" value="10u"/>
-<part name="C21" library="STEVES_BU" deviceset="CAPS" device="0603S" value="0.1u"/>
-<part name="C20" library="STEVES_BU" deviceset="CAPS" device="0603S" value="0.1u"/>
+<part name="C19" library="rcl" deviceset="C-EU" device="C1206" value="10"/>
+<part name="C18" library="rcl" deviceset="C-EU" device="C1206" value="10"/>
+<part name="C21" library="STEVES_BU" deviceset="CAPS" device="0603S" value="0.1"/>
+<part name="C20" library="STEVES_BU" deviceset="CAPS" device="0603S" value="0.1"/>
 <part name="C24" library="rcl" deviceset="C-EU" device="C1206" value="47"/>
 <part name="C26" library="rcl" deviceset="C-EU" device="C1206" value="47"/>
@@
 <part name="GND16" library="supply1" deviceset="GND" device=""/>
 <part name="GND22" library="supply1" deviceset="GND" device=""/>
+<part name="J9" library="STEVES_BU" deviceset="FCR7350G" device=""/>
+<part name="J10" library="STEVES_BU" deviceset="FCR7350G" device=""/>
+<part name="J11" library="STEVES_BU" deviceset="FCR7350G" device=""/>
+<part name="J12" library="STEVES_BU" deviceset="FCR7350G" device=""/>
 </parts>
 <sheets>
@@
 <attribute name="VALUE" x="187.96" y="187.96" size="1.778" layer="96" rot="MR270"/>
 </instance>
+<instance part="J9" gate="A" x="-66.04" y="160.02" rot="R180"/>
+<instance part="J10" gate="A" x="-66.04" y="147.32" rot="R180"/>
+<instance part="J11" gate="A" x="-66.04" y="134.62" rot="R180"/>
+<instance part="J12" gate="A" x="-66.04" y="121.92" rot="R180"/>
 </instances>
 <busses>

Commit message: EPGcontrol PCB updates - relay
Parts:
- added C17: 220n, STEVES_BU:CAPS0603S
- added C22: 150n, STEVES_BU:CAPS0603S
- added C25, C27: 10, STEVES_BU:CAPS1206S
- added D3, D4: DIODE, SparkFun-DiscreteSemi:DIODE-BAS16J
- added Q1, Q2: 2N3904, SparkFun-DiscreteSemi:TRANS_NPN-MMBT2222AL
- added R19, R20, R21, R22: 1K00, STEVES_BU:RESISTOR_SM0805S
Connections:
- removed net N$5: U1.!LDAC
- removed net N$9: U1.!CLR
- new net 5VD: C25.1, C27.1, R19.2, R20.2
- new net ADCSYNC: U$1.GP22, U2.!SYNC!/!RESET
- new net DACCS: U$1.GP13, U1.!SYNC
- new net DACRST: U$1.GP15, U1.!CLR
- new net LDAC: U$1.GP14, U1.!LDAC
- new net N$2: C17.1, U2.CAP
- new net N$3: Q2.B, R21.1
- new net R6: R21.2, U$1.GP27/A1
- new net R7: R22.2, U$1.GP26/A0
- new net RGND: Q1.E, Q2.E
- net ADCCLK: now also U$1.GP21
- net ADCRDY: now also U$1.GP20
- net AGND: now also C22.2
- net GND: now also C17.2
- net K6N: now also D4.A, Q2.C
- net K6P: now also C27.2, D4.C, R20.1
- net K7N: now also D3.A, Q1.C
- net K7P: now also C25.2, D3.C, R19.1
- net N$10: now also C22.1
- net N$4: now also Q1.B, R22.1; no longer U1.!SYNC
