File: hardware/pcb/eagle/EPGcontrolBipDAC.brd (EAGLE design)
At the start: 228.6 x 92.5 mm, 75 parts, among them J1 54-00248, J10 FCR7350G, J11 FCR7350G, J12 FCR7350G, J2 54-00248, J3 54-00248, J4 54-00248, J5 54-00248, J6 54-00248, J7 54-00248, J8 54-00248, J9 FCR7350G, Q1 600mA/40V, Q2 600mA/40V, U2 ADS131M08QPBSRQ1, U3 LTC2666CUH-16PBF, U4 TPS7A470X, U5 TPS7A33

Commit message: controller updates
Parts:
- removed C22: 150n, STEVES_BU:0603S
- added C28: 0.1, STEVES_BU:0603S
- added C29, C30: 1, STEVES_BU:0805S
- added C31: .01, STEVES_BU:0805S
Connections:
- removed net IOVCC: U3.18
- removed net N$10: C22.1
- removed net N$5: U$1.17
- removed net N$6: U$1.20
- removed net N$7: U$1.19
- removed net VCC: U3.28
- new net 3V3D: U$1.36, U3.17, U3.18, U3.28, U3.32
- new net DACRST: U$1.19, U3.24
- new net N$11: C31.1, U3.25
- new net N$8: C28.1, U3.26
- net -5V0: now also C30.1, U3.33
- net 5V0: now also C29.1
- net AGND: now also C28.2, C29.2, C30.2, C31.2, U3.1, U3.10, U3.11, U3.27, U3.29, U3.31; no longer C22.2
- net DACCS: now also U$1.20
Routing:
- net DACCS: track 0.00 -> 35.6 mm, vias 0 -> 2
- net SPIORX: track 11.1 -> 40.6 mm, vias 0 -> 2
- net -5V0: track 288.3 -> 310.6 mm, vias 1 -> 2
- net N$6: track 21.0 -> 0.00 mm, vias 1 -> 0
- net SPIOCLK: track 30.6 -> 50.3 mm, vias 1 -> 2
- net AGND: track 37.8 -> 55.1 mm, vias 14 -> 20
- net SPIOTX: track 33.4 -> 49.7 mm, vias 1 -> 2
- net VS7: track 80.1 -> 89.2 mm
- net VS4: track 23.3 -> 14.7 mm
- net VS1: track 70.0 -> 78.3 mm
- net VS3: track 18.1 -> 25.0 mm
- net 3V3D: track 0.00 -> 6.45 mm
- net VS5: track 30.6 -> 36.9 mm
- net VS6: track 68.6 -> 63.7 mm
- net VS0: track 95.4 -> 100.0 mm
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