File: hardware/pcb/eagle/EPGcontrolBipDAC.sch (EAGLE design)
At the start: 75 parts, among them J1 54-00248, J10 FCR7350G, J11 FCR7350G, J12 FCR7350G, J2 54-00248, J3 54-00248, J4 54-00248, J5 54-00248, J6 54-00248, J7 54-00248, J8 54-00248, J9 FCR7350G, Q1 600mA/40V, Q2 600mA/40V, U2 ADS131M08QPBSRQ1, U3 LTC2666CUH-16PBF, U4 TPS7A470X, U5 TPS7A33

Commit message: controller updates
Parts:
- removed C22: 150n, STEVES_BU:CAPS0603S
- added C28: 0.1, STEVES_BU:CAPS0603S
- added C29, C30: 1, STEVES_BU:CAPS0805S
- added C31: .01, STEVES_BU:CAPS0805S
Connections:
- removed net N$10: C22.1
- removed net N$5: U$1.GP13
- removed net N$6: U$1.GP15
- removed net N$7: U$1.GP14
- new net 3V3D: U$1.3V3OUT, U3.IOVCC, U3.MSP1, U3.TGP, U3.VCC
- new net DACRST: U$1.GP14, U3.!CLR
- new net N$11: C31.1, U3.REF
- new net N$8: C28.1, U3.REFCOMP
- net -5V0: now also C30.1, U3.EPAD
- net 5V0: now also C29.1
- net AGND: now also C28.2, C29.2, C30.2, C31.2, U3.GND, U3.GND_2, U3.MSP0, U3.MSP2, U3.REFLO, U3.REFLO_2; no longer C22.2
- net DACCS: now also U$1.GP15
